File: hardware/pcb/output/ADLFO.kicad_sch (KiCad schematic)
At the start: 114 parts, among them J1 TRIG1, J10 TRIG4, J11 CV4, J12 OUT4, J13 EURORACK 2x5 keyed, J14 OLED SSD1306 128x64, J2 CV1, J3 OUT1, J4 TRIG2, J5 CV2, J6 OUT2, J7 TRIG3, J8 CV3, J9 OUT3, Q1 MMBT3904, Q2 MMBT3904, Q3 MMBT3904, Q4 MMBT3904, SW1 CH 1, SW2 CH 2, SW3 CH 3, SW4 CH 4, U1 Daisy Seed (socketed), U2 MCP4728-E/UN, U3 MCP6004-I/SL, U4 TL074CDR, U5 R-78E5.0-0.5

Commit message: Adapt PCB placement to 20 HP with Adafruit DAC module and Eurorack power provisions
Parts:
- added C10: 47uF 10V low ESR candidate, ADLFO:radial_cap, symbol ADLFO:C10
- added C11: 100nF, ADLFO:c0805, symbol ADLFO:C11
- added C12: 100nF, ADLFO:c0805, symbol ADLFO:C12
- added F1: PTC 0.5A hold candidate, ADLFO:ptc1812, symbol ADLFO:F1
- added RP11: 10k DNP, ADLFO:r0805, symbol ADLFO:RP11
- added RP12: 10k DNP, ADLFO:r0805, symbol ADLFO:RP12
- added RP13: 10k DNP, ADLFO:r0805, symbol ADLFO:RP13
- added RP14: 10k DNP, ADLFO:r0805, symbol ADLFO:RP14
- added RP21: 10k DNP, ADLFO:r0805, symbol ADLFO:RP21
- added RP22: 10k DNP, ADLFO:r0805, symbol ADLFO:RP22
- added RP23: 10k DNP, ADLFO:r0805, symbol ADLFO:RP23
- added RP24: 10k DNP, ADLFO:r0805, symbol ADLFO:RP24
- added RP31: 10k DNP, ADLFO:r0805, symbol ADLFO:RP31
- added RP32: 10k DNP, ADLFO:r0805, symbol ADLFO:RP32
- added RP33: 10k DNP, ADLFO:r0805, symbol ADLFO:RP33
- added RP34: 10k DNP, ADLFO:r0805, symbol ADLFO:RP34
- added RP41: 10k DNP, ADLFO:r0805, symbol ADLFO:RP41
- added RP42: 10k DNP, ADLFO:r0805, symbol ADLFO:RP42
- added RP43: 10k DNP, ADLFO:r0805, symbol ADLFO:RP43
- added RP44: 10k DNP, ADLFO:r0805, symbol ADLFO:RP44
- R1, R2: value 4.7k -> 4.7k DNP
- U2: value MCP4728-E/UN -> Adafruit MCP4728 STEMMA QT breakout; footprint ADLFO:msop10 -> ADLFO:mcp4728_breakout
Connections:
- net +12V_IN: now also F1.1; no longer D1.2
- net +3V3: now also U2.12 (JP2_VCC), C12.1, RP11.1, RP12.1, RP13.1, RP14.1, RP21.1, RP22.1, RP23.1, RP24.1, RP31.1, RP32.1, RP33.1, RP34.1, RP41.1, RP42.1, RP43.1, RP44.1
- net +5V_SEED: now also C10.1, C11.1
- net D0: now also RP11.2
- net D1: now also RP12.2
- net D10: now also RP41.2
- net D11: now also U2.3 (JP1_SCL); no longer U2.2 (SCL)
- net D12: now also U2.4 (JP1_SDA); no longer U2.3 (SDA)
- net D13: now also RP42.2
- net D14: now also RP43.2
- net D2: now also RP13.2
- net D24: now also RP24.2
- net D25: now also RP14.2
- net D26: now also RP34.2
- net D27: now also RP44.2
- net D3: now also RP21.2
- net D4: now also RP22.2
- net D5: now also RP23.2
- net D7: now also RP31.2
- net D8: now also RP32.2
- net D9: now also RP33.2
- net DAC1: now also U2.8 (JP2_VA); no longer U2.6 (VA)
- net DAC2: now also U2.9 (JP2_VB); no longer U2.7 (VB)
- net DAC3: now also U2.10 (JP2_VC); no longer U2.8 (VC)
- net DAC4: now also U2.11 (JP2_VD); no longer U2.9 (VD)
- net GND: now also U2.2 (JP1_GND), U2.5 (JP1_LDAC), U2.7 (JP2_GND), C10.2, C11.2, C12.2; no longer U2.10 (VSS), U2.4 (LDAC)
- new net +12V_FUSED: D1.2, F1.2
Other:
- title: ADLFO REV A — electrical placement draft -> ADLFO REV B — electrical placement draft
