File: hardware/pcb/output/Adolfo-panel.kicad_pcb (KiCad board)
At the start: 2 copper layers, 96.2 x 110.5 mm, 26 parts, among them J1 IN1 PJ398SM, J10 IN4 PJ398SM, J11 CTRL4 PJ398SM, J12 OUT4 PJ398SM, J14 SSD1306 breakout raised, J2 CTRL1 PJ398SM, J3 OUT1 PJ398SM, J4 IN2 PJ398SM, J5 CTRL2 PJ398SM, J6 OUT2 PJ398SM, J7 IN3 PJ398SM, J8 CTRL3 PJ398SM, J9 OUT3 PJ398SM, K1 6x6 tact height TBD, K2 6x6 tact height TBD, K3 6x6 tact height TBD, K4 6x6 tact height TBD

Commit message: fix(pcb): harden 20hp carrier and center panel display
Complete rev D schematics, routed boards and native KiCad checks.
Fix input normals, reset latch, fault resistor ratings and via placement.
Center the OLED module and window; update routing and mechanical exports.
Record supply sequencing, 5 V supervision and converter backend blockers.

Validation: 2027 CAD checks, zero ERC/DRC violations, host and SPICE tests.
Parts:
- removed JP: Panel link 2x20 candidate, ADOLFO:header40
- added J15: Samtec SSW-120-02-G-D, ADOLFO:socket40, B.Cu at (50.6, 87.0)
- E1, E2, E3, E4: value EC11 click candidate -> ALPS EC11E18244AU
- J14: value SSD1306 breakout raised -> Waveshare 0.96inch OLED Module (D), I2C; footprint ADOLFO:oled -> ADOLFO:oled7
- K1, K2, K3, K4: value 6x6 tact height TBD -> E-Switch TL1105DF160Q
- moved J14 26.6 mm to (50.6, 11.0)
- renumbered REF** to H1, REF** to H2, REF** to H3, REF** to H4
Connections:
- J1 pad TN: (no net) -> GND
- J10 pad TN: (no net) -> GND
- J11 pad TN: (no net) -> unconnected-(J11-TIP_NORMAL-PadTN)
- J12 pad TN: (no net) -> unconnected-(J12-TIP_NORMAL-PadTN)
- J14 pad 1: GND -> +3V3
- J14 pad 2: +3V3 -> GND
- J14 pad 3: I2C_SCL -> I2C_SDA
- J14 pad 4: I2C_SDA -> I2C_SCL
- J2 pad TN: (no net) -> unconnected-(J2-TIP_NORMAL-PadTN)
- J3 pad TN: (no net) -> unconnected-(J3-TIP_NORMAL-PadTN)
- J4 pad TN: (no net) -> GND
- J5 pad TN: (no net) -> unconnected-(J5-TIP_NORMAL-PadTN)
- J6 pad TN: (no net) -> unconnected-(J6-TIP_NORMAL-PadTN)
- J7 pad TN: (no net) -> GND
- J8 pad TN: (no net) -> unconnected-(J8-TIP_NORMAL-PadTN)
- J9 pad TN: (no net) -> unconnected-(J9-TIP_NORMAL-PadTN)
Routing:
- net GND: track 0.00 -> 542.6 mm
- net OLED_RESET: track 0.00 -> 124.0 mm, vias 0 -> 1
- net I2C_SCL: track 0.00 -> 97.9 mm
- net I2C_SDA: track 0.00 -> 94.3 mm
- net +3V3: track 0.00 -> 94.1 mm
- net ENC4_CLICK: track 0.00 -> 70.4 mm, vias 0 -> 1
- net ENC1_B: track 0.00 -> 65.9 mm, vias 0 -> 1
- net ENC1_A: track 0.00 -> 65.6 mm, vias 0 -> 1
- net KEY1: track 0.00 -> 62.7 mm, vias 0 -> 1
- net ENC4_A: track 0.00 -> 59.2 mm, vias 0 -> 1
- net ENC4_B: track 0.00 -> 58.1 mm, vias 0 -> 1
- net KEY4: track 0.00 -> 57.9 mm, vias 0 -> 1
- net KEY3: track 0.00 -> 53.8 mm, vias 0 -> 1
- net OUT1: track 0.00 -> 49.6 mm
- net ENC2_A: track 0.00 -> 49.6 mm, vias 0 -> 1
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Other:
- rule pad_to_mask_clearance: 0.0 -> 0
